File: scsi/scsi.kicad_pcb (KiCad board)
At the start: 2 copper layers, 100 x 90 mm, 22 parts, among them J1 SCSI, J2 VAMPIRE_OR_HBA, J3 ENABLE_TERMINATION, J4 CPU, U1 AM33C93

Commit message: Final Board Design as of First Manufacture - V1.0
Parts:
- removed the REF** at (114.5, 34.1)
- removed the REF** at (32.4, 105.7)
- removed the REF** at (115.3, 112.4)
- moved ? 27.2 mm to (59.6, 105.8)
- moved ? 8.11 mm to (106.5, 35.4)
- moved ? 2.30 mm to (113.8, 110.7)
- moved REF** 1.36 mm to (30.9, 34.5)
Routing:
- net Net-(J1-Pin_44): vias 3 -> 2
- net GND: vias 7 -> 0
